File: kicad/ev-charger-met16.sch (KiCad schematic (older format))
At the start: 57 parts, among them J1 Screw_Terminal_01x02, J10 Conn_02x02_Counter_Clockwise, J2 Conn_01x03, J3 Conn_01x15, J4 Conn_01x15, J5 Lusterklemme-6mm2-40A, J6 Lusterklemme-6mm2-40A, J7 LCD-Sure, J8 UART-Harwin4, J9 Conn_01x03, SW1 SW_PT65-501, SW2 SW_DPDT_x2, U1 ARDUINO-NANO, U2 HLK-PM01, U3 ebay-253052736386, U4 ACS712, U6 AD822

Commit message: Redesign v0.3 finished, gerber-files ready for print production
Parts:
- removed SW2: SW_DPDT_x2, MyFootprints:SW-ebay-171865305033, symbol SW_DPDT_x2
- added C13, C17: 1u, Capacitors_SMD:C_1206_HandSoldering, symbol C
- added C14: 220n, Capacitors_SMD:C_1206_HandSoldering, symbol C
- added C15, C16: 100n, Capacitors_SMD:C_1206_HandSoldering, symbol C
- added D7: blau, LEDs:LED_PLCC-2, symbol LED
- added D8, D9: D_Schottky, Diodes_SMD:D_SMA_Handsoldering, symbol D_Schottky
- added J12, J13: Conn_01x01, Project:Solder_via_5x5_forWire4mm2, symbol Conn_01x01
- added K1: Omron_G5RL-1-E, Relays_THT:Relay_DPDT_Panasonic_JW2, symbol Omron_G5RL-1-E
- added K2: Conn_01x02, Pin_Headers:Pin_Header_Straight_1x02_Pitch2.54mm, symbol Conn_01x02
- added Q1, Q2: FDV303N, TO_SOT_Packages_SMD:SOT-23_Handsoldering, symbol BSS138
- added R36: 560R, Resistors_SMD:R_1206_HandSoldering, symbol R
- added R37, R39: 47k, Resistors_SMD:R_1206_HandSoldering, symbol R
- R10: value 10k -> 100M
- R13, R26: value 10k -> 1k
- R14, R15: value 2k7 -> 560R
- R16, R18, R23, R24: value 0R -> 47k
- R21: value 39k -> 27k
- R22: value 15k -> 10k
- R29: value 3k3 -> 47k
- R31: value 1k -> 15k
- R32: value 22k -> 100M
- R33: value 100k -> 120k
- R34: value 10k -> 33k
- R35: value 10k -> 3k3
Connections:
- net labels added: LOUT
- wire segments 245 -> 293
- no-connect marks 5 -> 6
Other:
- note added: "Fotek SSR 100A Relais"
- note added: "LED L on Arduino Nano\n= PB5 (D13)"
- note added: "R10 optional"
- note added: "R22 optional"
- moved on the sheet: C10, C11, C12, C6, C7, C8, D1, D2, D3, D5, J1, J10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
