File: kicad/voltage-sensor.sch (KiCad schematic (older format))
At the start: 18 parts, among them T1 Transformer_1P_1S, U5 LM358

Commit message: Redesign v0.3 finished, gerber-files ready for print production
Parts:
- RV1: value 10k -> 100k
Connections:
- net +5V: now also R3.2
- net at R11.1, T1.3 (SA): now also R3.1, R8.2, U5.5 (+); no longer R3.2
Other:
- moved on the sheet: C1, C3, C4, C5, R1, R2, R3, R4, R6, R7, R8, R9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
