File: kicad/ev-charger-met16.kicad_pcb (KiCad board)
At the start: 2 copper layers, 165 x 70 mm, 83 parts, among them J1 Screw_Terminal_01x02, J10 Conn_02x02_Counter_Clockwise, J2 Conn_01x03, J3 Conn_01x15, J4 Conn_01x15, J5 Lusterklemme-6mm2-40A, J6 Lusterklemme-6mm2-40A, J7 LCD-Sure, J8 UART-Harwin4, J9 Conn_01x03, SW1 SW_PT65-501, SW2 SW_DPDT_x2, T1 Transformer_1P_1S, U1 ARDUINO-NANO, U2 HLK-PM01, U3 ebay-253052736386, U4 ACS712, U5 LM358, U6 AD822

Commit message: Redesign v0.3 finished, gerber-files ready for print production
Parts:
- removed SW2: SW_DPDT_x2, MyFootprints:SW-ebay-171865305033
- added C13: 1u, Capacitors_SMD:C_1206_HandSoldering, B.Cu at (128.8, 91.9)
- added C14: 220n, Capacitors_SMD:C_1206_HandSoldering, B.Cu at (119.8, 67.1)
- added C15: 100n, Capacitors_SMD:C_1206_HandSoldering, B.Cu at (128.8, 94.1)
- added C16: 100n, Capacitors_SMD:C_1206_HandSoldering, B.Cu at (96.6, 69.5)
- added C17: 1u, Capacitors_SMD:C_1206_HandSoldering, B.Cu at (94.5, 69.5)
- added D7: blau, LEDs:LED_PLCC-2, F.Cu at (202.3, 79.6)
- added D8: D_Schottky, Diodes_SMD:D_SMA_Handsoldering, B.Cu at (113.7, 65.0)
- added D9: D_Schottky, Diodes_SMD:D_SMA_Handsoldering, F.Cu at (139.6, 92.1)
- added J11: Conn_01x02, Pin_Headers:Pin_Header_Straight_1x02_Pitch2.54mm, F.Cu at (121.3, 61.3)
- added J12: Conn_01x01, Project:Solder_via_5x5_forWire4mm2, F.Cu at (128.0, 119.0)
- added J13: Conn_01x01, Project:Solder_via_5x5_forWire4mm2, F.Cu at (147.5, 121.0)
- added K1: Omron_G5RL-1-E, Relays_THT:Relay_DPDT_Panasonic_JW2, F.Cu at (134.0, 97.0)
- added Q1: FDV303N, TO_SOT_Packages_SMD:SOT-23_Handsoldering, F.Cu at (113.3, 60.5)
- added Q2: FDV303N, TO_SOT_Packages_SMD:SOT-23_Handsoldering, F.Cu at (146.3, 90.4)
- added R36: 560R, Resistors_SMD:R_1206_HandSoldering, F.Cu at (199.3, 84.8)
- added R37: 47k, Resistors_SMD:R_1206_HandSoldering, F.Cu at (105.9, 59.9)
- added R39: 47k, Resistors_SMD:R_1206_HandSoldering, F.Cu at (151.9, 88.8)
- R10: value 10k -> 100M
- R13, R26: value 10k -> 1k
- R14, R15: value 2k7 -> 560R
- R16, R18, R23, R24: value 0R -> 47k
- R21: value 39k -> 27k
- R22: value 15k -> 10k
- R29: value 3k3 -> 47k
- R31: value 1k -> 15k
- R32: value 22k -> 100M
- R33: value 100k -> 120k
- R34: value 10k -> 33k
- R35: value 10k -> 3k3
- RV1: value 10k -> 100k
- moved R14 31.8 mm to (207.0, 82.9), turned to 180 degrees
- moved D2 18.3 mm to (207.8, 79.6), turned to 0 degrees
- moved R30 12.4 mm to (115.1, 96.6)
- moved C6 12.2 mm to (117.6, 96.6)
- moved C7 9.07 mm to (131.2, 102.5), turned to 0 degrees
- moved C5 7.85 mm to (141.1, 86.6)
- moved D4 7.17 mm to (206.0, 58.9)
- moved R12 6.91 mm to (102.9, 83.6)
- moved R6 5.61 mm to (129.3, 82.0)
- moved D3 5.34 mm to (205.6, 63.0)
- moved U5 4.98 mm to (142.5, 81.9)
- moved R7 4.93 mm to (145.5, 77.2)
- moved R9 4.78 mm to (151.9, 83.4)
- moved C3 4.73 mm to (149.6, 83.4)
- moved R4 3.28 mm to (141.1, 89.0)
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Connections:
- J6 pad 3: /L -> /LOUT
- R14 pad 2: /A4 -> /A5
- R3 pad 1: Net-(R3-Pad1) -> Net-(R11-Pad1)
- R3 pad 2: Net-(R11-Pad1) -> +5V
- R34 pad 1: +5V -> Net-(R34-Pad1)
- R34 pad 2: Net-(R34-Pad2) -> +5V
- R35 pad 1: Net-(R34-Pad2) -> Net-(R34-Pad1)
- R5 pad 1: /CP -> Net-(R32-Pad2)
- R5 pad 2: Net-(R32-Pad2) -> /CP
- R8 pad 2: Net-(R3-Pad1) -> Net-(R11-Pad1)
- U5 pad 5: Net-(R3-Pad1) -> Net-(R11-Pad1)
- U6 pad 2: Net-(R34-Pad2) -> Net-(R34-Pad1)
Routing:
- net +5V: track 163.0 -> 271.1 mm, vias 5 -> 11
- net /A5: track 34.6 -> 122.2 mm, vias 0 -> 2
- net /A4: track 6.70 -> 66.2 mm, vias 0 -> 2
- net Net-(D2-Pad2): track 44.8 -> 3.41 mm, vias 2 -> 0
- net GND: track 91.6 -> 125.4 mm, vias 7 -> 10
- net Net-(R3-Pad1): track 32.7 -> 0.00 mm, vias 1 -> 0
- net Net-(R11-Pad1): track 9.98 -> 36.5 mm, vias 0 -> 1
- net Net-(R34-Pad1): track 0.00 -> 22.5 mm, vias 0 -> 2
- net Net-(R34-Pad2): track 22.5 -> 0.00 mm, vias 2 -> 0
- net +12V: track 12.0 -> 25.9 mm
- net Net-(D9-Pad2): track 0.00 -> 12.7 mm
- net Net-(D8-Pad2): track 0.00 -> 12.5 mm, vias 0 -> 1
- net /L: track 78.9 -> 86.0 mm
- net /PE: track 57.7 -> 51.1 mm
- net /N: track 61.7 -> 55.4 mm, vias 1 -> 0
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- added copper zone on B.Cu, net /L
- added copper zone on B.Cu, net /LOUT
- removed copper zone on F.Cu, net /L
Other:
- board text added: "7A...16A"
- board text added: "EV Charger MET16 V0.3 / SX"
- board text added: "L (IN)"
- board text added: "L (OUT)"
- board text added: "L(IN)"
- board text added: "L(OUT)"
- board text removed: "7A ... 16A"
- board text removed: "EV Charger MET16 V0.2 / SX"
- board text removed: "L"
- board text removed: "OFF"
- board text removed: "ON"

Commit message: update project settings
Parts:
- renumbered J11 to K2
Routing:
- net GND: track 125.4 -> 138.9 mm, vias 10 -> 18
- net /CP: track 96.0 -> 97.9 mm, vias 2 -> 4
- net /MCURR: track 33.5 -> 34.5 mm
- net Net-(D9-Pad2): track 12.7 -> 13.2 mm
Other:
- board text added: "+12V"
- board text added: "0V"
- board text added: "K1"
- board text added: "LCD"
- board text added: "Life LED"
- board text added: "SSR"
- board text added: "SSR(100A)"
- board text added: "SSR-1"
- board text added: "SSR-2"
- board text added: "SSR-3"
- board text added: "SSR-4"
- board text added: "UART 5V"
